Commit message: fix: define lidar position xacro properties

File: src/lio_sam_move_base_tutorial/robot_gazebo/scout_gazebo/urdf/base_no_realsense.xacro (robot description, xacro)
@@ -30,4 +30,6 @@
     <!-- VLP16 激光雷达 -->
     <xacro:include filename="$(find scout_gazebo)/urdf/laser_support.xacro" />
+    <xacro:property name="lidar_x" value="${support_x_size}" />
+    <xacro:property name="lidar_z" value="${support_z_size + support_length/2}" />
     <xacro:include filename="$(find velodyne_description)/urdf/VLP-16.urdf.xacro"/>
     <xacro:VLP-16 parent="support" name="velodyne" topic="/velodyne_points" organize_cloud="${organize_cloud}" hz="$(arg lidar_hz)" samples="$(arg lidar_samples)" gpu="${gpu}">
