Commit message: chore: sync workspace

File: src/lio_sam_move_base_tutorial/robot_gazebo/scout_gazebo/urdf/base.xacro (robot description, xacro)
@@ -16,4 +16,8 @@
     <xacro:arg name="organize_cloud" default="true"/>
     <xacro:property name="organize_cloud" value="$(arg organize_cloud)" />
+    <xacro:arg name="lidar_hz" default="10"/>
+    <xacro:arg name="lidar_samples" default="440"/>
+    <xacro:arg name="use_skid_steer" default="false"/>
+    <xacro:arg name="use_planar_move" default="true"/>
     <material name="black">
         <color rgba="0.0 0.0 0.0 1.0" />
@@ -33,5 +37,5 @@
     <xacro:include filename="$(find scout_gazebo)/urdf/laser_support.xacro" />
     <xacro:include filename="$(find velodyne_description)/urdf/VLP-16.urdf.xacro"/>
-    <xacro:VLP-16 parent="support" name="velodyne" topic="/velodyne_points" organize_cloud="${organize_cloud}" hz="10" samples="440" gpu="${gpu}">
+    <xacro:VLP-16 parent="support" name="velodyne" topic="/velodyne_points" organize_cloud="${organize_cloud}" hz="$(arg lidar_hz)" samples="$(arg lidar_samples)" gpu="${gpu}">
           <origin xyz="0 0 ${support_length/2}" rpy="0 0 0" />
     </xacro:VLP-16>

File: src/lio_sam_move_base_tutorial/robot_gazebo/scout_gazebo/urdf/base_no_realsense.xacro (robot description, xacro)
@@ -19,4 +19,6 @@
     <xacro:arg name="lidar_hz" default="10"/>
     <xacro:arg name="lidar_samples" default="440"/>
+    <xacro:arg name="use_skid_steer" default="false"/>
+    <xacro:arg name="use_planar_move" default="true"/>
     <material name="black">
         <color rgba="0.0 0.0 0.0 1.0" />
@@ -30,4 +32,6 @@
     <!-- VLP16 激光雷达 -->
     <xacro:include filename="$(find scout_gazebo)/urdf/laser_support.xacro" />
+    <xacro:property name="lidar_x" value="${support_x_size}" />
+    <xacro:property name="lidar_z" value="${support_z_size + support_length/2}" />
     <xacro:include filename="$(find velodyne_description)/urdf/VLP-16.urdf.xacro"/>
     <xacro:VLP-16 parent="support" name="velodyne" topic="/velodyne_points" organize_cloud="${organize_cloud}" hz="$(arg lidar_hz)" samples="$(arg lidar_samples)" gpu="${gpu}">

File: src/lio_sam_move_base_tutorial/robot_gazebo/scout_gazebo/urdf/laser_support.xacro (robot description, xacro)
@@ -2,7 +2,8 @@
 <robot name="laser_support" xmlns:xacro="http://wiki.ros.org/xacro">
     <!-- 雷达支架 -->
-    <xacro:property name="support_length" value="0.30" /> <!-- 支架长度 -->
+    <!-- NOTE: These values must match the static TF in pcd_gazebo_world/launch/orchard_pcd_sim.launch -->
+    <xacro:property name="support_length" value="0.48502" /> <!-- 支架长度 -->
     <xacro:property name="support_radius" value="0.025" /> <!-- 支架半径 -->
-    <xacro:property name="support_x_size" value="-0.2" /> <!-- 支架安装的x坐标 -->
+    <xacro:property name="support_x_size" value="0.175" /> <!-- 支架安装的x坐标 -->
     <xacro:property name="support_y_size" value="0.0" /> <!-- 支架安装的y坐标 -->
     <xacro:property name="support_z_size" value="${base_z_size}" /> <!-- 支架安装的z坐标:底盘高度 / 2 + 支架高度 / 2  -->

File: src/lio_sam_move_base_tutorial/robot_gazebo/scout_gazebo/urdf/move.xacro (robot description, xacro)
@@ -1,4 +1,9 @@
 <?xml version="1.0"?>
 <robot name="my_car_move" xmlns:xacro="http://wiki.ros.org/xacro">
+    <!-- Drive plugin selection:
+         - Enabling BOTH skid_steer + planar_move at the same time will cause the robot to "乱跑".
+         - Default: planar_move only. -->
+    <xacro:property name="use_skid_steer" value="$(arg use_skid_steer)" />
+    <xacro:property name="use_planar_move" value="$(arg use_planar_move)" />
     <!-- 传动实现:用于连接控制器与关节 -->
     <xacro:macro name="joint_trans" params="joint_name">
@@ -21,28 +26,36 @@
     <xacro:joint_trans joint_name="rear_right_wheel" />
     <!-- 控制器 -->
-    <gazebo>
-  		<plugin name="skid_steer_drive_controller" filename="libgazebo_ros_skid_steer_drive.so">
-    		<updateRate>100.0</updateRate>
-    		<robotNamespace>/</robotNamespace>
-    		<leftFrontJoint>front_left_wheel</leftFrontJoint>
-    		<rightFrontJoint>front_right_wheel</rightFrontJoint>
-    		<leftRearJoint>rear_left_wheel</leftRearJoint>
-    		<rightRearJoint>rear_right_wheel</rightRearJoint>
-    		<wheelSeparation>${track}</wheelSeparation>
-    		<wheelDiameter>${wheel_radius * 2}</wheelDiameter>
-    		<robotBaseFrame>base_link</robotBaseFrame>
-    		<torque>20</torque>
-    		<topicName>cmd_vel</topicName>
-    		<broadcastTF>false</broadcastTF>
-  		</plugin>
-	</gazebo>
-  <gazebo>
-    <plugin name="object_controller" filename="libgazebo_ros_planar_move.so">
-      <commandTopic>cmd_vel</commandTopic>
-      <odometryTopic>odom</odometryTopic>
-      <odometryFrame>odom</odometryFrame>
-      <odometryRate>20.0</odometryRate>
-      <robotBaseFrame>base_link</robotBaseFrame>
-    </plugin>
-  </gazebo>
+    <xacro:if value="${use_skid_steer}">
+        <gazebo>
+            <plugin name="skid_steer_drive_controller" filename="libgazebo_ros_skid_steer_drive.so">
+                <updateRate>100.0</updateRate>
+                <robotNamespace>/</robotNamespace>
+                <leftFrontJoint>front_left_wheel</leftFrontJoint>
+                <rightFrontJoint>front_right_wheel</rightFrontJoint>
+                <leftRearJoint>rear_left_wheel</leftRearJoint>
+                <rightRearJoint>rear_right_wheel</rightRearJoint>
+                <wheelSeparation>${track}</wheelSeparation>
+                <wheelDiameter>${wheel_radius * 2}</wheelDiameter>
+                <robotBaseFrame>base_link</robotBaseFrame>
+                <torque>200</torque>
+                <commandTopic>cmd_vel</commandTopic>
+                <odometryTopic>odom</odometryTopic>
+                <odometryFrame>odom</odometryFrame>
+                <broadcastTF>true</broadcastTF>
+            </plugin>
+        </gazebo>
+    </xacro:if>
+    <xacro:unless value="${use_skid_steer}">
+        <xacro:if value="${use_planar_move}">
+            <gazebo>
+                <plugin name="object_controller" filename="libgazebo_ros_planar_move.so">
+                    <commandTopic>cmd_vel</commandTopic>
+                    <odometryTopic>odom</odometryTopic>
+                    <odometryFrame>odom</odometryFrame>
+                    <odometryRate>20.0</odometryRate>
+                    <robotBaseFrame>base_link</robotBaseFrame>
+                </plugin>
+            </gazebo>
+        </xacro:if>
+    </xacro:unless>
 </robot>

File: src/lio_sam_move_base_tutorial/robot_gazebo/scout_gazebo/urdf/scout_wheel_type1.xacro (robot description, xacro)
@@ -48,5 +48,5 @@
             <child link="${wheel_prefix}_wheel_link"/>
             <xacro:insert_block name="joint_pose"/>
-            <axis xyz="0 -1 0" rpy="0 0 0" />
+            <axis xyz="0 1 0" rpy="0 0 0" />
         </joint>
     </xacro:macro>

File: src/lio_sam_move_base_tutorial/robot_gazebo/scout_gazebo/urdf/scout_wheel_type2.xacro (robot description, xacro)
@@ -48,5 +48,5 @@
             <child link="${wheel_prefix}_wheel_link"/>
             <xacro:insert_block name="joint_pose"/>
-            <axis xyz="0 -1 0" rpy="0 0 0" />
+            <axis xyz="0 1 0" rpy="0 0 0" />
         </joint>
     </xacro:macro>
